File: Motor_Control/stepper_controller_pcb/stepper_controller_pcb.kicad_pcb (KiCad board)
At the start: 2 copper layers, 42.9 x 54 mm, 11 parts, among them J1 Conn_02x03_Odd_Even, J2 Conn_01x02_Pin, J3 Conn_01x04, J4 Conn_01x04, J5 Conn_01x04_Pin

Commit message: autotracker works
Parts:
- added J6: Conn_01x02_Pin, Connector_PinHeader_2.54mm:PinHeader_1x02_P2.54mm_Vertical, F.Cu at (103.6, 83.0)
- added J7: Conn_01x03, Connector_JST:JST_XH_B3B-XH-A_1x03_P2.50mm_Vertical, F.Cu at (88.8, 62.0)
- added J8: Conn_01x03, Connector_JST:JST_XH_B3B-XH-A_1x03_P2.50mm_Vertical, F.Cu at (112.9, 62.0)
- moved REF** 47.4 mm to (80.6, 119.0)
- moved J1 47.1 mm to (108.5, 117.5)
- moved J3 47.1 mm to (116.0, 93.5)
- moved J4 47.1 mm to (116.0, 106.0)
- moved R1 47.1 mm to (103.2, 91.9)
- moved A1 47.1 mm to (84.5, 76.8)
- moved J2 47.1 mm to (109.5, 82.5)
- moved J5 47.1 mm to (115.0, 75.2)
- moved REF** 47.1 mm to (119.9, 119.0)
- moved REF** 38.3 mm to (80.6, 62.0)
- moved REF** 38.0 mm to (119.9, 62.1)
Connections:
- A1 pad 10: unconnected-(A1-D7-Pad10) -> LASER_PWM
- A1 pad 28: unconnected-(A1-~{RESET}-Pad28) -> RST!
- R1 pad 2: ENA_ -> ENA
Routing:
- net ENA_: track 114.4 -> 0.00 mm
- net gnd!: track 12.7 -> 126.7 mm
- net LASER_PWM: track 0.00 -> 65.0 mm
- net +12V: track 0.00 -> 24.1 mm
- net ENA: track 26.3 -> 40.9 mm
- net +5V: track 98.1 -> 106.5 mm
- net RST!: track 0.00 -> 4.49 mm
- net DIR_Y: track 40.7 -> 41.5 mm
Other:
- board size 42.9 x 54 mm -> 45.9 x 63.5 mm
