File: Motor_Control/stepper_controller_pcb/stepper_controller_pcb.kicad_sch (KiCad schematic)
At the start: 7 parts, among them J1 Conn_02x03_Odd_Even, J2 Conn_01x02_Pin, J3 Conn_01x04, J4 Conn_01x04, J5 Conn_01x04_Pin

Commit message: autotracker works
Parts:
- added J6: Conn_01x02_Pin, Connector_PinHeader_2.54mm:PinHeader_1x02_P2.54mm_Vertical, symbol Connector:Conn_01x02_Pin
- added J7, J8: Conn_01x03, Connector_JST:JST_XH_B3B-XH-A_1x03_P2.50mm_Vertical, symbol Connector_Generic:Conn_01x03
Connections:
- net gnd!: now also J6.1 (Pin_1), J7.2 (Pin_2), J8.2 (Pin_2)
- net LASER_PWM: now reaches A1.10 (D7)
- net LASER_PWM: now also J7.3 (Pin_3), J8.3 (Pin_3)
- net RST!: now reaches A1.28 (~{RESET})
- net RST!: now also J6.2 (Pin_2)
- new net +12V: J7.1 (Pin_1), J8.1 (Pin_1)
Other:
- moved on the sheet: A1, J1, J2, J3, J4, J5, R1
